File: pcb/tanfolyamrobot.brd (EAGLE design)
At the start: 81.3 x 58.7 mm, 78 parts, among them IC1 STM32F10XRXT6, IC2 7805, IC4 FT232RL, IC5 LD117AS33TR, M1 DRV8833, Q2 BSS123, Q3 BSS123, Q4 BSS123, X1 CSTCE08M, X2 PWR, X6 KUSBVX-BS1N

Commit message: cosmetic changes (#1)
Connections:
- net N$3 renamed ESP_CHPD
Routing:
- net +5V/1: track 43.0 -> 48.8 mm
- net +3V3: track 244.8 -> 242.0 mm
- net ESP_CHPD: track 10.3 -> 12.2 mm
Changed lines of the file:
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@@
 <via x="52.705" y="43.18" extent="1-16" drill="0.35"/>
 <wire x1="63.5" y1="46.99" x2="61.595" y2="48.895" width="0.3048" layer="16"/>
-<wire x1="55.245" y1="48.895" x2="61.595" y2="48.895" width="0.3048" layer="16"/>
 <wire x1="52.705" y1="43.18" x2="51.015" y2="43.18" width="0.3048" layer="1"/>
 <contactref element="U$1" pad="VCC"/>
@@
 <wire x1="44.03" y1="31.535" x2="41.91" y2="31.535" width="0.2032" layer="1"/>
 <via x="44.45" y="31.115" extent="1-16" drill="0.35"/>
-<wire x1="44.45" y1="31.115" x2="45.72" y2="32.385" width="0.3048" layer="16"/>
-<wire x1="45.72" y1="38.1" x2="49.8475" y2="42.2275" width="0.3048" layer="16"/>
-<wire x1="49.8475" y1="42.2275" x2="50.8" y2="43.18" width="0.3048" layer="16"/>
-<wire x1="45.72" y1="32.385" x2="45.72" y2="38.1" width="0.3048" layer="16"/>
+<wire x1="45.72" y1="32.385" x2="44.45" y2="31.115" width="0.3048" layer="16"/>
 <wire x1="65.14" y1="36.645" x2="65.14" y2="37.73" width="0.3048" layer="1"/>
 <wire x1="65.405" y1="46.355" x2="64.77" y2="46.99" width="0.3048" layer="1"/>
@@
 <wire x1="63.5" y1="40.64" x2="65.405" y2="42.545" width="0.3048" layer="1"/>
 <wire x1="65.405" y1="42.545" x2="65.405" y2="46.355" width="0.3048" layer="1"/>
-<wire x1="50.8" y1="44.45" x2="50.8" y2="43.18" width="0.3048" layer="16"/>
-<wire x1="52.705" y1="43.18" x2="50.8" y2="43.18" width="0.3048" layer="16"/>
-<wire x1="50.8" y1="44.45" x2="55.245" y2="48.895" width="0.3048" layer="16"/>
 <wire x1="45.07" y1="5.095" x2="45.1625" y2="5.095" width="0.3048" layer="16"/>
 <wire x1="40.005" y1="6.35" x2="43.815" y2="6.35" width="0.3048" layer="16"/>
@@
 <wire x1="47.625" y1="19.685" x2="48.895" y2="18.415" width="0.3048" layer="1"/>
 <wire x1="48.895" y1="18.415" x2="48.895" y2="15.24" width="0.3048" layer="1"/>
-<via x="47.625" y="15.24" extent="1-16" drill="0.35"/>
-<wire x1="47.625" y1="17.78" x2="44.45" y2="20.955" width="0.3048" layer="16"/>
+<via x="48.895" y="18.415" extent="1-16" drill="0.35"/>
 <wire x1="44.45" y1="31.115" x2="44.45" y2="26.035" width="0.3048" layer="16"/>
-<wire x1="44.45" y1="26.035" x2="44.45" y2="20.955" width="0.3048" layer="16"/>
-<wire x1="47.625" y1="17.78" x2="47.625" y2="15.24" width="0.3048" layer="16"/>
+<wire x1="44.45" y1="26.035" x2="44.45" y2="22.86" width="0.3048" layer="16"/>
 <contactref element="R10" pad="2"/>
 <wire x1="31.535" y1="24.13" x2="31.535" y2="24.765" width="0.2032" layer="1"/>
@@
 <wire x1="35.56" y1="22.225" x2="36.83" y2="20.955" width="0.3048" layer="1"/>
 <wire x1="36.83" y1="20.955" x2="36.83" y2="19.685" width="0.3048" layer="1"/>
-<wire x1="47.625" y1="15.24" x2="48.895" y2="15.24" width="0.3048" layer="1"/>
 <wire x1="31.006140625" y1="26.600865625" x2="31.006140625" y2="26.561140625" width="0.2032" layer="1"/>
 <wire x1="31.006140625" y1="26.561140625" x2="30.48" y2="26.035" width="0.2032" layer="1"/>
@@
 <wire x1="33.97885" y1="47.93615" x2="32.385" y2="49.53" width="0.3048" layer="16"/>
 <wire x1="32.385" y1="49.53" x2="24.13" y2="49.53" width="0.3048" layer="16"/>
-<wire x1="33.97885" y1="47.93615" x2="44.13885" y2="47.93615" width="0.3048" layer="16"/>
-<wire x1="44.13885" y1="47.93615" x2="49.8475" y2="42.2275" width="0.3048" layer="16"/>
+<wire x1="44.45" y1="22.86" x2="48.895" y2="18.415" width="0.3048" layer="16"/>
+<wire x1="45.72" y1="32.385" x2="45.72" y2="38.7477" width="0.3048" layer="16"/>
+<wire x1="33.97885" y1="47.93615" x2="45.72" y2="47.93615" width="0.3048" layer="16"/>
+<wire x1="45.72" y1="38.7477" x2="48.895" y2="41.9227" width="0.3048" layer="16"/>
+<wire x1="48.895" y1="44.76115" x2="45.72" y2="47.93615" width="0.3048" layer="16"/>
+<wire x1="48.895" y1="41.9227" x2="48.895" y2="43.18" width="0.3048" layer="16"/>
+<wire x1="48.895" y1="43.18" x2="48.895" y2="44.76115" width="0.3048" layer="16"/>
+<wire x1="52.705" y1="43.18" x2="48.895" y2="43.18" width="0.3048" layer="16"/>
+<wire x1="53.02885" y1="48.895" x2="48.895" y2="44.76115" width="0.3048" layer="16"/>
+<wire x1="61.595" y1="48.895" x2="53.02885" y2="48.895" width="0.3048" layer="16"/>
 </signal>
 <signal name="SWD_SWO">
@@
 <contactref element="C8" pad="1"/>
 <contactref element="IC4" pad="17"/>
-<wire x1="56.134" y1="31.027" x2="59.143" y2="31.027" width="0.3048" layer="1"/>
-<wire x1="59.94" y1="30.23" x2="59.94" y2="29.395" width="0.3048" layer="1"/>
-<wire x1="59.143" y1="31.027" x2="59.94" y2="30.23" width="0.3048" layer="1"/>
+<wire x1="56.134" y1="31.027" x2="59.298575" y2="31.027" width="0.3048" layer="1"/>
+<wire x1="59.94" y1="30.385575" x2="59.94" y2="29.395" width="0.3048" layer="1"/>
+<wire x1="59.298575" y1="31.027" x2="59.94" y2="30.385575" width="0.3048" layer="1"/>
 </signal>
 <signal name="USB_DM_FTDI">
@@
 <contactref element="R3" pad="2"/>
 <wire x1="63.84" y1="29.395" x2="63.84" y2="28.235" width="0.2032" layer="1"/>
-<wire x1="64.77" y1="27.305" x2="64.77" y2="26.67" width="0.2032" layer="1"/>
-<wire x1="65.363725" y1="26.076275" x2="66.206" y2="26.076275" width="0.2032" layer="1"/>
-<wire x1="63.84" y1="28.235" x2="64.77" y2="27.305" width="0.2032" layer="1"/>
-<wire x1="64.77" y1="26.67" x2="65.363725" y2="26.076275" width="0.2032" layer="1"/>
+<wire x1="63.84" y1="28.235" x2="64.135" y2="27.94" width="0.2032" layer="1"/>
+<wire x1="64.135" y1="27.94" x2="65.405" y2="27.94" width="0.2032" layer="1"/>
+<wire x1="66.206" y1="27.139" x2="66.206" y2="26.076275" width="0.2032" layer="1"/>
+<wire x1="65.405" y1="27.94" x2="66.206" y2="27.139" width="0.2032" layer="1"/>
 </signal>
 <signal name="FTDI_RXLEDN">
@@
 <contactref element="R4" pad="2"/>
 <wire x1="63.19" y1="29.395" x2="63.19" y2="28.094425" width="0.2032" layer="1"/>
-<wire x1="63.19" y1="28.094425" x2="64.135" y2="27.149425" width="0.2032" layer="1"/>
+<wire x1="63.19" y1="28.094425" x2="64.77" y2="26.514425" width="0.2032" layer="1"/>
 <wire x1="65.408175" y1="24.126825" x2="66.2314" y2="24.126825" width="0.2032" layer="1"/>
-<wire x1="64.135" y1="27.149425" x2="64.135" y2="25.4" width="0.2032" layer="1"/>
-<wire x1="64.135" y1="25.4" x2="65.408175" y2="24.126825" width="0.2032" layer="1"/>
+<wire x1="64.77" y1="26.514425" x2="64.77" y2="24.765" width="0.2032" layer="1"/>
+<wire x1="64.77" y1="24.765" x2="65.408175" y2="24.126825" width="0.2032" layer="1"/>
 </signal>
 <signal name="FTDI_RTSN">
@@
 <wire x1="43.815" y1="10.1854" x2="42.2402" y2="8.6106" width="0.2032" layer="16"/>
 </signal>
-<signal name="N$3">
+<signal name="ESP_CHPD">
 <contactref element="U$1" pad="CH_PD"/>
 <contactref element="C18" pad="1"/>
@@
 <wire x1="44.87" y1="19.685" x2="43.815" y2="19.685" width="0.2032" layer="1"/>
 <wire x1="43.815" y1="19.685" x2="43.815" y2="11.5225" width="0.2032" layer="1"/>
-<wire x1="43.815" y1="11.5225" x2="45.1625" y2="10.175" width="0" layer="19" extent="1-1"/>
+<wire x1="43.815" y1="11.5225" x2="45.1625" y2="10.175" width="0.2032" layer="1"/>
 </signal>
 <signal name="PA6">
@@
 <contactref element="LED2" pad="A"/>
 <contactref element="R27" pad="1"/>
-<via x="69.215" y="19.685" extent="1-16" drill="0.35"/>
-<wire x1="69.215" y1="19.685" x2="69.173725" y2="19.726275" width="0.2032" layer="16"/>
-<wire x1="69.173725" y1="31.22385" x2="69.173725" y2="19.726275" width="0.2032" layer="16"/>
-<wire x1="69.215" y1="19.685" x2="69.215" y2="10.16" width="0.2032" layer="16"/>
+<via x="72.856725" y="20.799425" extent="1-16" drill="0.35"/>
+<wire x1="72.856725" y1="20.799425" x2="69.173725" y2="24.482425" width="0.2032" layer="16"/>
+<wire x1="69.173725" y1="31.22385" x2="69.173725" y2="24.482425" width="0.2032" layer="16"/>
 <via x="69.215" y="10.16" extent="1-16" drill="0.35"/>
 <wire x1="74.181" y1="8.255" x2="71.12" y2="8.255" width="0.4064" layer="1"/>
@@
 <wire x1="66.675" y1="10.675" x2="68.7" y2="10.675" width="0.4064" layer="1"/>
 <wire x1="76.36" y1="10.434" x2="74.181" y2="8.255" width="0.4064" layer="1"/>
-<wire x1="69.215" y1="19.685" x2="69.215" y2="20.84" width="0.2032" layer="1"/>
 <wire x1="70.993" y1="20.84" x2="69.215" y2="20.84" width="0.2032" layer="1"/>
 <wire x1="63.08" y1="24.003" x2="64.106425" y2="24.003" width="0.2032" layer="1"/>
 <wire x1="67.269425" y1="20.84" x2="69.215" y2="20.84" width="0.2032" layer="1"/>
 <wire x1="64.106425" y1="24.003" x2="67.269425" y2="20.84" width="0.2032" layer="1"/>
+<wire x1="78.105" y1="12.179" x2="76.36" y2="10.434" width="0.2032" layer="1"/>
+<wire x1="78.105" y1="12.179" x2="78.105" y2="17.145" width="0.2032" layer="1"/>
+<wire x1="74.450575" y1="20.799425" x2="72.856725" y2="20.799425" width="0.2032" layer="1"/>
+<wire x1="78.105" y1="17.145" x2="74.450575" y2="20.799425" width="0.2032" layer="1"/>
+<wire x1="70.993" y1="20.84" x2="72.81615" y2="20.84" width="0.2032" layer="1"/>
+<wire x1="72.81615" y1="20.84" x2="72.856725" y2="20.799425" width="0.2032" layer="1"/>
 </signal>
 </signals>
