File: pcb/v3/tanfolyamrobot.kicad_sch (KiCad schematic)
At the start: 77 parts, among them IC2 LP2950?CDT, IC4 FT232RL, IC5 LD117A?S, M1 DRV8833, Q1 BSO201SP, Q2 BSS123, Q3 BSS123, Q4 BSS123, SW1 SW_DPDT_x2, U1 STM32F411RCTx, X1 MURATA_CSTCE, X2 1751248, X6 KUSBVX-BS1N

Commit message: Fixed issues on schematic
Connections:
- net FTDI_BOOT0_OUT renamed FTDI_CBUS2
- no-connect marks 15 -> 26
Other:
- moved on the sheet: R5
Changed lines of the file:
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@@
 	)
 	(junction
-		(at 372.11 119.38)
-		(diameter 0)
-		(color 0 0 0 0)
-	)
-	(junction
 		(at 345.44 43.18)
 		(diameter 0)
@@
 	)
 	(no_connect
+		(at 429.26 111.76)
+	)
+	(no_connect
+		(at 429.26 162.56)
+	)
+	(no_connect
 		(at 170.18 246.38)
 	)
 	(no_connect
+		(at 429.26 172.72)
+	)
+	(no_connect
+		(at 393.7 124.46)
+	)
+	(no_connect
 		(at 170.18 251.46)
 	)
@@
 	)
 	(no_connect
+		(at 429.26 121.92)
+	)
+	(no_connect
 		(at 491.49 69.85)
 	)
 	(no_connect
+		(at 429.26 104.14)
+	)
+	(no_connect
+		(at 429.26 124.46)
+	)
+	(no_connect
 		(at 491.49 62.23)
 	)
 	(no_connect
+		(at 393.7 142.24)
+	)
+	(no_connect
 		(at 142.24 251.46)
 	)
 	(no_connect
+		(at 393.7 144.78)
+	)
+	(no_connect
+		(at 429.26 109.22)
+	)
+	(no_connect
 		(at 525.78 134.62)
 	)
@@
 	)
 	(no_connect
+		(at 81.28 330.2)
+	)
+	(no_connect
 		(at 170.18 271.78)
 	)
@@
 	(wire
 		(pts
-			(xy 513.08 266.7) (xy 447.04 266.7)
-		)
-		(stroke
-			(width 0.1524)
-			(type solid)
-		)
-	)
-	(wire
-		(pts
 			(xy 208.28 83.82) (xy 208.28 76.2)
 		)
@@
 	(wire
 		(pts
-			(xy 378.46 106.68) (xy 378.46 119.38)
+			(xy 378.46 106.68) (xy 378.46 123.19)
 		)
 		(stroke
@@
 	(wire
 		(pts
-			(xy 513.08 264.16) (xy 447.04 264.16)
-		)
-		(stroke
-			(width 0.1524)
-			(type solid)
-		)
-	)
-	(wire
-		(pts
 			(xy 170.18 266.7) (xy 195.58 266.7)
 		)
@@
 	(wire
 		(pts
-			(xy 513.08 243.84) (xy 447.04 243.84)
-		)
-		(stroke
-			(width 0.1524)
-			(type solid)
-		)
-	)
-	(wire
-		(pts
 			(xy 492.76 302.26) (xy 492.76 297.18)
 		)
@@
 	(wire
 		(pts
-			(xy 513.08 248.92) (xy 447.04 248.92)
-		)
-		(stroke
-			(width 0.1524)
-			(type solid)
-		)
-	)
-	(wire
-		(pts
 			(xy 480.06 241.3) (xy 513.08 241.3)
 		)
@@
 	(wire
 		(pts
-			(xy 381 241.3) (xy 416.56 241.3)
+			(xy 447.04 243.84) (xy 513.08 243.84)
+		)
+		(stroke
+			(width 0.1524)
+			(type solid)
+		)
+	)
+	(wire
+		(pts
+			(xy 381 241.3) (xy 421.64 241.3)
+		)
+		(stroke
+			(width 0.1524)
+			(type solid)
+		)
+	)
+	(wire
+		(pts
+			(xy 447.04 261.62) (xy 513.08 261.62)
 		)
 		(stroke
@@
 	(wire
 		(pts
+			(xy 447.04 269.24) (xy 513.08 269.24)
+		)
+		(stroke
+			(width 0.1524)
+			(type solid)
+		)
+	)
+	(wire
+		(pts
 			(xy 55.88 269.24) (xy 55.88 246.38)
 		)
@@
 	(wire
 		(pts
+			(xy 447.04 266.7) (xy 513.08 266.7)
+		)
+		(stroke
+			(width 0.1524)
+			(type solid)
+		)
+	)
+	(wire
+		(pts
 			(xy 480.06 49.53) (xy 491.49 49.53)
 		)
@@
 	(wire
 		(pts
-			(xy 513.08 269.24) (xy 447.04 269.24)
-		)
-		(stroke
-			(width 0.1524)
-			(type solid)
-		)
-	)
-	(wire
-		(pts
 			(xy 83.82 325.12) (xy 83.82 327.66)
 		)
@@
 	(wire
 		(pts
+			(xy 372.11 119.38) (xy 372.11 123.19)
+		)
+		(stroke
+			(width 0)
+			(type default)
+		)
+	)
+	(wire
+		(pts
 			(xy 119.38 50.8) (xy 167.64 50.8)
 		)
@@
 	(wire
 		(pts
-			(xy 355.6 246.38) (xy 335.28 246.38)
+			(xy 447.04 248.92) (xy 513.08 248.92)
 		)
 		(stroke
@@
 	(wire
 		(pts
-			(xy 487.68 142.24) (xy 487.68 134.62)
+			(xy 355.6 246.38) (xy 335.28 246.38)
 		)
 		(stroke
@@
 	(wire
 		(pts
-			(xy 342.9 353.06) (xy 335.28 353.06)
+			(xy 487.68 142.24) (xy 487.68 134.62)
 		)
 		(stroke
@@
 	(wire
 		(pts
-			(xy 177.8 327.66) (xy 170.18 327.66)
+			(xy 342.9 353.06) (xy 335.28 353.06)
 		)
 		(stroke
@@
 	(wire
 		(pts
-			(xy 139.7 279.4) (xy 139.7 289.56)
+			(xy 177.8 327.66) (xy 170.18 327.66)
 		)
 		(stroke
@@
 	(wire
 		(pts
-			(xy 210.82 342.9) (xy 210.82 353.06)
+			(xy 139.7 279.4) (xy 139.7 289.56)
 		)
 		(stroke
@@
 	(wire
 		(pts
-			(xy 372.11 119.38) (xy 372.11 118.11)
+			(xy 210.82 342.9) (xy 210.82 353.06)
 		)
 		(stroke
-			(width 0)
-			(type default)
+			(width 0.1524)
+			(type solid)
 		)
 	)
@@
 	(wire
 		(pts
-			(xy 170.18 243.84) (xy 195.4276 243.84)
+			(xy 170.18 243.84) (xy 195.58 243.84)
 		)
 		(stroke
@@
 	(wire
 		(pts
-			(xy 429.26 162.56) (xy 445.77 162.56)
-		)
-		(stroke
-			(width 0)
-			(type default)
-		)
-	)
-	(wire
-		(pts
 			(xy 154.94 342.9) (xy 154.94 353.06)
 		)
@@
 	(wire
 		(pts
-			(xy 492.76 274.32) (xy 492.76 276.86)
+			(xy 492.76 274.32) (xy 492.76 275.59)
 		)
 		(stroke
@@
 	(wire
 		(pts
-			(xy 513.08 261.62) (xy 447.04 261.62)
+			(xy 492.76 285.75) (xy 492.76 287.02)
 		)
 		(stroke
-			(width 0.1524)
-			(type solid)
+			(width 0)
+			(type default)
 		)
 	)
@@
 	(wire
 		(pts
-			(xy 378.46 119.38) (xy 372.11 119.38)
+			(xy 378.46 123.19) (xy 372.11 123.19)
 		)
 		(stroke
@@
 	(wire
 		(pts
+			(xy 447.04 264.16) (xy 513.08 264.16)
+		)
+		(stroke
+			(width 0.1524)
+			(type solid)
+		)
+	)
+	(wire
+		(pts
 			(xy 93.98 327.66) (xy 114.3 327.66)
 		)
@@
 	)
 	(label "COLOR_OUT"
-		(at 421.64 360.68 0)
+		(at 436.88 360.68 0)
 		(effects
 			(font
@@
 	)
 	(label "LCD_RST"
-		(at 449.58 243.84 0)
+		(at 447.04 243.84 0)
 		(effects
 			(font
@@
 	)
 	(label "LCD_D5"
-		(at 449.58 264.16 0)
+		(at 447.04 264.16 0)
 		(effects
 			(font
@@
 	)
 	(label "LCD_EN"
-		(at 449.58 248.92 0)
+		(at 447.04 248.92 0)
 		(effects
 			(font
@@
 	)
 	(label "LCD_D7"
-		(at 449.58 269.24 0)
+		(at 447.04 269.24 0)
 		(effects
 			(font
@@
 	)
 	(label "LCD_D4"
-		(at 449.58 261.62 0)
+		(at 447.04 261.62 0)
 		(effects
 			(font
@@
 	)
 	(label "COLOR_S2"
-		(at 421.64 358.14 0)
+		(at 436.88 358.14 0)
 		(effects
 			(font
@@
 		)
 	)
-	(label "FTDI_BOOT0_OUT"
-		(at 201.93 134.62 0)
-		(effects
-			(font
-				(size 1.2446 1.2446)
-			)
-			(justify left bottom)
-		)
-	)
 	(label "SERVO"
 		(at 464.82 342.9 0)
@@
 	)
 	(label "FTDI_RTSN"
-		(at 195.4276 243.84 0)
+		(at 195.58 243.84 0)
 		(effects
 			(font
@@
 	)
 	(label "MOTOR_FAULTN"
-		(at 396.24 241.3 0)
+		(at 421.64 241.3 0)
 		(effects
 			(font
@@
 	)
 	(label "LCD_D6"
-		(at 449.58 266.7 0)
+		(at 447.04 266.7 0)
 		(effects
 			(font
@@
 	)
 	(label "COLOR_S3"
-		(at 421.64 355.6 0)
+		(at 436.88 355.6 0)
 		(effects
 			(font
@@
 	(symbol
 		(lib_id "tanfolyamrobot-eagle-import:R-EU_R0603")
-		(at 492.76 281.94 90)
+		(at 492.76 280.67 90)
 		(unit 1)
 		(exclude_from_sim no)
@@
 		(dnp no)
 		(property "Reference" "R5"
-			(at 491.2614 285.75 0)
+			(at 491.236 282.448 0)
 			(effects
 				(font
@@
 		)
 		(property "Value" "R-EU_R0603"
-			(at 496.062 285.75 0)
+			(at 496.062 284.48 0)
 			(effects
 				(font
@@
 		)
 		(property "Footprint" "tanfolyamrobot:R0603"
-			(at 492.76 281.94 0)
+			(at 492.76 280.67 0)
 			(effects
 				(font
@@
 		)
 		(property "Datasheet" ""
-			(at 492.76 281.94 0)
+			(at 492.76 280.67 0)
 			(effects
 				(font
@@
 		)
 		(property "Description" ""
-			(at 492.76 281.94 0)
+			(at 492.76 280.67 0)
 			(effects
 				(font

Commit message: Finishing touches
Parts:
- added C20: 4u7, tanfolyamrobot:C0603, symbol tanfolyamrobot-eagle-import:C-EUC0603
- added C21, C24: 100n, tanfolyamrobot:C0603, symbol tanfolyamrobot-eagle-import:C-EUC0603
- added C22, C23: 10u, tanfolyamrobot:C0805K, symbol tanfolyamrobot-eagle-import:C-EUC0805K
- added C25, C26: 68u, tanfolyamrobot:B_3528-21R, symbol tanfolyamrobot-eagle-import:CPOL-EUB/3528-21R
- added FB1: 220, Inductor_SMD:L_0603_1608Metric, symbol Device:FerriteBead
- added R13: 10K, tanfolyamrobot:R0603, symbol tanfolyamrobot-eagle-import:R-EU_R0603
- added R14: 4K7, tanfolyamrobot:R0603, symbol tanfolyamrobot-eagle-import:R-EU_R0603
- D3, D4, D6: footprint tanfolyamrobot:MICROMELF-W -> Diode_SMD:D_SOD-323F
- RX0, TX0: footprint tanfolyamrobot:CHIP-LED0603 -> LED_SMD:LED_0603_1608Metric
Connections:
- net +3V3: now also C20.1, C23.1, C26.+, FB1.2, R13.2; no longer U1.13 (VDDA)
- net +5V: now also C25.+
- net +5V/1: now also RX0.2, TX0.2; no longer RX0.A, TX0.A
- net BOOT: now also D3.1; no longer D3.C
- net BUTTON: now also R13.1
- net FTDI_CBUS2: now also D3.2; no longer D3.A
- net FTDI_RTSN: now also D4.1; no longer D4.C
- net GND: now also C20.2, C21.2, C22.2, C23.2, C24.2, C25.-, C26.-
- net RSTN: now also D4.2, D6.2; no longer D4.A, D6.A
- net SWD_RSTN: now also D6.1; no longer D6.C
- net VCC_SENSE: now also R14.2; no longer U1.21 (PA5)
- net at R3.1: now also TX0.1; no longer TX0.C
- net at R4.1: now also RX0.1; no longer RX0.C
- new net: C22.1, C24.1, FB1.1, U1.13 (VDDA)
- new net VCC_SENSE_FILTERED: C21.1, R14.1, U1.21 (PA5)
Other:
- note added: "2:3 voltage deviders are there to protect the 3V3 uC from the 5V sygnals of the encoders."
- note added: "Pullups and capacitors are inside the module."
- note removed: "VBAT VDDA VSSA"
- moved on the sheet: C1, C10, C11, C12, C13, C14, C2, C3, C4, C7, IC2, IC5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

Commit message: Known issues and fixes
Other:
- note added: "Ismert problémák és javításuk: - FTDI-n keresztüli feltöltés nem megy ha PB2 nincs földrekötve. -> PU helyett PD ellenállás. - PB12 boot módban reseteli az FTDI chipet, megszakítva a feltöltést. -> Vagy más pinen kell power detect, vagy el kell hagyni teljesen, vagy kölön feszültségosztó kell neki."
Changed lines of the file:
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@@
 		)
 	)
+	(text "Ismert problémák és javításuk:\n - FTDI-n keresztüli feltöltés nem megy ha PB2 nincs földrekötve. ->\n    PU helyett PD ellenállás.\n - PB12 boot módban reseteli az FTDI chipet, megszakítva a feltöltést. ->\n    Vagy más pinen kell power detect, vagy el kell hagyni teljesen, vagy kölön feszültségosztó kell neki."
+		(exclude_from_sim no)
+		(at 5.842 -34.29 0)
+		(effects
+			(font
+				(size 7.62 7.62)
+				(color 255 0 0 1)
+			)
+			(justify left)
+		)
+	)
 	(text "Notes:\n- BUTTON's pin must be pulled up internally\n- US_TRIG must be operated as open drain output\n- MOTOR_FAULTN must be pulled up internally"
 		(exclude_from_sim no)
@@
 					(unit 1)
 				)
+			)
+		)
+	)
+	(symbol
+		(lib_id "tanfolyamrobot-eagle-import:A4L-LOC")
+		(at 287.02 198.12 0)
+		(unit 1)
+		(exclude_from_sim no)
+		(in_bom yes)
+		(on_board yes)
+		(dnp no)
+		(property "Reference" "#FRAME3"
+			(at 287.02 198.12 0)
+			(effects
+				(font
+					(size 1.27 1.27)
+				)
+				(hide yes)
+			)
+		)
+		(property "Value" "A4L-LOC"
+			(at 287.02 198.12 0)
+			(effects
+				(font
+					(size 1.27 1.27)
+				)
+				(hide yes)
+			)
+		)
+		(property "Footprint" ""
+			(at 287.02 198.12 0)
+			(effects
+				(font
+					(size 1.27 1.27)
+				)
+				(hide yes)
+			)
+		)
+		(property "Datasheet" ""
+			(at 287.02 198.12 0)
+			(effects
+				(font
+					(size 1.27 1.27)
+				)
+				(hide yes)
+			)
+		)
+		(property "Description" ""
+			(at 287.02 198.12 0)
+			(effects
+				(font
+					(size 1.27 1.27)
+				)
+			)
+		)
+		(instances
+			(project "tanfolyamrobot"
+				(path "/6a846de4-0b89-4d79-a2ed-e6fc99adef94"
+					(reference "#FRAME3")
+					(unit 1)
+				)
